Commit message: Simple sim with laser scanner to grab pose of enemy robot. Attempt to integrate with EKF not yet successful

File: interfearence-description/urdf/diff_interfearence.urdf (robot description, URDF)
Before this commit: robot interfearence, 4 links, 3 joints
Links:
- added link hokuyo, mass 0.0; visual box size=0.05 0.05 0.07
Joints:
- added joint hokuyo_joint: type fixed, parent chassis, child hokuyo, origin xyz=0 0 0.035

File: interfearence-description/urdf/interfearence.urdf (robot description, URDF)
Before this commit: robot interfearence, 4 links, 3 joints
Links:
- added link hokuyo, mass 0.0; visual box size=0.05 0.05 0.07
- link chassis: geometry collision box size=0.195 0.195 0.05; visual box size=0.195 0.195 0.05
Joints:
- added joint hokuyo_joint: type fixed, parent chassis, child hokuyo, origin xyz=0 0 0.035
