Commit message: Created working arena edge detection message and plugins for gazebo

File: interfearence-description/urdf/cad_interfearence.urdf.xacro (robot description, xacro)
@@ -75,4 +75,28 @@
   </link>
   <gazebo reference="front_left_line_sensor">
+    <sensor name="front_left_line_sensor_sensor" type="camera">
+      <camera name="front_left_camera">
+        <image>
+          <width>1</width>
+          <height>1</height>
+          <format>R8G8B8</format>
+        </image>
+        <clip>
+          <near>0.002</near>
+        </clip>
+      </camera>
+      <plugin name="front_left_edge_detector_plugin"
+              filename="libarena_edge_detection_plugin.so">
+        <cameraName>front_left_camera</cameraName>
+        <alwaysOn>true</alwaysOn>
+        <updateRate>30</updateRate>
+        <imageTopicName>rgb/image_raw</imageTopicName>
+        <cameraInfoTopicName>rgb/camera_info</cameraInfoTopicName>
+        <frameName>/$(arg robotns)/front_left_line_sensor</frameName>
+        <topicName>/$(arg robotns)/edge_sensors/front_left</topicName>
+        <upperThreshhold>0.5</upperThreshhold>
+        <lowerThreshhold>0.4</lowerThreshhold>
+      </plugin>
+    </sensor>
     <material>Gazebo/Red</material>
   </gazebo>
@@ -101,4 +125,28 @@
   </link>
   <gazebo reference="front_right_line_sensor">
+    <sensor name="front_right_line_sensor_sensor" type="camera">
+      <camera name="front_right_camera">
+        <image>
+          <width>1</width>
+          <height>1</height>
+          <format>R8G8B8</format>
+        </image>
+        <clip>
+          <near>0.002</near>
+        </clip>
+      </camera>
+      <plugin name="front_right_edge_detector_plugin"
+              filename="libarena_edge_detection_plugin.so">
+        <cameraName>front_right_camera</cameraName>
+        <alwaysOn>true</alwaysOn>
+        <updateRate>30</updateRate>
+        <imageTopicName>rgb/image_raw</imageTopicName>
+        <cameraInfoTopicName>rgb/camera_info</cameraInfoTopicName>
+        <frameName>/$(arg robotns)/front_right_line_sensor</frameName>
+        <topicName>/$(arg robotns)/edge_sensors/front_right</topicName>
+        <upperThreshhold>0.5</upperThreshhold>
+        <lowerThreshhold>0.4</lowerThreshhold>
+      </plugin>
+    </sensor>
     <material>Gazebo/Red</material>
   </gazebo>
@@ -275,5 +323,5 @@
     <parent link="base_footprint"/>
     <child link="hokuyo"/>
-    <origin rpy="0 0 -1.57" xyz="-8.000e-05 -3.485e-02  2.744e-02"/>
+    <origin rpy="0 -0.02 -1.57" xyz="-8.000e-05 -3.485e-02  2.744e-02"/>
   </joint>
   <link name="rear_right_line_sensor">
@@ -295,5 +343,29 @@
     </visual>
   </link>
-  <gazebo reference="rear_left_line_sensor">
+  <gazebo reference="rear_right_line_sensor">
+    <sensor name="rear_right_line_sensor_sensor" type="camera">
+      <camera name="rear_right_camera">
+        <image>
+          <width>1</width>
+          <height>1</height>
+          <format>R8G8B8</format>
+        </image>
+        <clip>
+          <near>0.002</near>
+        </clip>
+      </camera>
+      <plugin name="rear_right_edge_detector_plugin"
+              filename="libarena_edge_detection_plugin.so">
+        <cameraName>rear_right_camera</cameraName>
+        <alwaysOn>true</alwaysOn>
+        <updateRate>30</updateRate>
+        <imageTopicName>rgb/image_raw</imageTopicName>
+        <cameraInfoTopicName>rgb/camera_info</cameraInfoTopicName>
+        <frameName>/$(arg robotns)/rear_right_line_sensor</frameName>
+        <topicName>/$(arg robotns)/edge_sensors/rear_right</topicName>
+        <upperThreshhold>0.5</upperThreshhold>
+        <lowerThreshhold>0.4</lowerThreshhold>
+      </plugin>
+    </sensor>
     <material>Gazebo/Red</material>
   </gazebo>
@@ -321,5 +393,29 @@
     </visual>
   </link>
-  <gazebo reference="rear_right_line_sensor">
+  <gazebo reference="rear_left_line_sensor">
+    <sensor name="rear_left_line_sensor_sensor" type="camera">
+      <camera name="rear_left_camera">
+        <image>
+          <width>1</width>
+          <height>1</height>
+          <format>R8G8B8</format>
+        </image>
+        <clip>
+          <near>0.002</near>
+        </clip>
+      </camera>
+      <plugin name="rear_left_edge_detector_plugin"
+              filename="libarena_edge_detection_plugin.so">
+        <cameraName>rear_left_camera</cameraName>
+        <alwaysOn>true</alwaysOn>
+        <updateRate>30</updateRate>
+        <imageTopicName>rgb/image_raw</imageTopicName>
+        <cameraInfoTopicName>rgb/camera_info</cameraInfoTopicName>
+        <frameName>/$(arg robotns)/rear_left_line_sensor</frameName>
+        <topicName>/$(arg robotns)/edge_sensors/rear_left</topicName>
+        <upperThreshhold>0.5</upperThreshhold>
+        <lowerThreshhold>0.4</lowerThreshhold>
+      </plugin>
+    </sensor>
     <material>Gazebo/Red</material>
   </gazebo>

Commit message: fixed front 2 sensors

File: interfearence-description/urdf/cad_interfearence.urdf.xacro (robot description, xacro)
@@ -97,6 +97,6 @@
         <frameName>/$(arg robotns)/front_left_line_sensor</frameName>
         <topicName>/$(arg robotns)/edge_sensors/front_left</topicName>
-        <upperThreshhold>0.5</upperThreshhold>
-        <lowerThreshhold>0.4</lowerThreshhold>
+        <upperThreshhold>0.52</upperThreshhold>
+        <lowerThreshhold>0.42</lowerThreshhold>
       </plugin>
     </sensor>
@@ -106,5 +106,5 @@
     <parent link="base_footprint"/>
     <child link="front_left_line_sensor"/>
-    <origin rpy="0 0 0" xyz="0.08972 -0.05966  0.00631"/>
+    <origin rpy="0 0 0" xyz="0.08972 -0.05966  0.000631"/>
   </joint>
   <link name="front_right_line_sensor">
@@ -147,6 +147,6 @@
         <frameName>/$(arg robotns)/front_right_line_sensor</frameName>
         <topicName>/$(arg robotns)/edge_sensors/front_right</topicName>
-        <upperThreshhold>0.5</upperThreshhold>
-        <lowerThreshhold>0.4</lowerThreshhold>
+        <upperThreshhold>0.52</upperThreshhold>
+        <lowerThreshhold>0.42</lowerThreshhold>
       </plugin>
     </sensor>
@@ -156,5 +156,5 @@
     <parent link="base_footprint"/>
     <child link="front_right_line_sensor"/>
-    <origin rpy="0 0 0" xyz="-0.08972 -0.05966  0.00631"/>
+    <origin rpy="0 0 0" xyz="-0.08972 -0.05966  0.000631"/>
   </joint>
   <link name="front_scoop">
@@ -180,5 +180,5 @@
     <mu2>0.2</mu2>
     <maxVel>0.0</maxVel>
-    <minDepth>0.001</minDepth>
+    <minDepth>0.0005</minDepth>
     <material>Gazebo/Gold</material>
   </gazebo>

Commit message: Robot finder update in progress - working on grouping points together.

File: interfearence-description/urdf/cad_interfearence.urdf.xacro (robot description, xacro)
@@ -325,5 +325,5 @@
     <parent link="base_footprint"/>
     <child link="hokuyo"/>
-    <origin rpy="0 -0.02 -1.57" xyz="-8.000e-05 -3.485e-02  2.744e-02"/>
+    <origin rpy="0 -0.03 -1.57" xyz="-8.000e-05 -3.485e-02  2.744e-02"/>
   </joint>
   <link name="rear_right_line_sensor">

Commit message: New controller ready to test - gazebo inertias need to be looked at?

File: interfearence-description/urdf/cad_interfearence.urdf.xacro (robot description, xacro)
@@ -192,5 +192,5 @@
       <mass value="0.31653412374925943"/>
       <origin rpy="0 0 0" xyz="0 0 0"/>
-      <inertia ixx="0.0014886350669894822" ixy="-0.0010718170567998425" ixz="-0.00041293261607713784" iyy="0.0013525795511995277" iyz="-0.0004689861809890939" izz="0.0023894152299137974"/>
+      <inertia ixx="0.0014886350669894822" ixy="-0.0" ixz="-0.0" iyy="0.0013525795511995277" iyz="-0.0" izz="0.0014886350669894822"/>
     </inertial>
     <collision name="left_wheel_collision">
@@ -232,5 +232,5 @@
       <mass value="0.3165346352615723"/>
       <origin rpy="0 0 0" xyz="0 0 0"/>
-      <inertia ixx="0.001488247009527325" ixy="0.0010716472878659678" ixz="0.00041292582180353995" iyy="0.0013525719181349898" iyz="-0.0004688703199637584" izz="0.0023890378944060355"/>
+      <inertia ixx="0.001488247009527325" ixy="0.0" ixz="0.0" iyy="0.0013525719181349898" iyz="-0.0" izz="0.001488247009527325"/>
     </inertial>
     <collision name="right_wheel_collision">

Commit message: Inertias and PIDs updated

File: interfearence-description/urdf/cad_interfearence.urdf.xacro (robot description, xacro)
@@ -9,4 +9,5 @@
       <!-- the launch file will replace this with something sensible -->
       <robotNamespace>$(arg robotns)</robotNamespace>
+      <robotSimType>gazebo_ros_control/DefaultRobotHWSim</robotSimType>
     </plugin>
     <!-- plugin to simulate the electromagnet -->
@@ -28,7 +29,7 @@
   <link name="base_footprint">
     <inertial>
-      <mass value="1.7923895668327776"/>
+      <mass value="2.4"/>
       <origin rpy="0 0 0" xyz="0.00178 0.02496 0.04945"/>
-      <inertia ixx="0.010567555781567964" ixy="5.0178754500137904e-05" ixz="-0.0002784618841121355" iyy="0.010348269788112794" iyz="-0.0024424380725769257" izz="0.007947774757175114"/>
+      <inertia ixx="0.016" ixy="0.0" ixz="0.0" iyy="0.016" iyz="0.0" izz="0.016"/>
     </inertial>
     <collision name="base_footprint_collision">
@@ -192,5 +193,5 @@
       <mass value="0.31653412374925943"/>
       <origin rpy="0 0 0" xyz="0 0 0"/>
-      <inertia ixx="0.0014886350669894822" ixy="-0.0" ixz="-0.0" iyy="0.0013525795511995277" iyz="-0.0" izz="0.0014886350669894822"/>
+      <inertia ixx="0.000122" ixy="-0.0" ixz="-0.0" iyy="0.000122" iyz="-0.0" izz="0.000137"/>
     </inertial>
     <collision name="left_wheel_collision">
@@ -226,5 +227,8 @@
       <hardwareInterface>hardware_interface/EffortJointInterface</hardwareInterface>
     </joint>
-    <actuator name="left_wheel_motor"/>
+    <actuator name="left_wheel_motor">
+      <hardwareInterface>hardware_interface/EffortJointInterface</hardwareInterface>
+      <mechanicalReduction>1</mechanicalReduction>
+    </actuator>
   </transmission>
   <link name="right_wheel">
@@ -232,5 +236,5 @@
       <mass value="0.3165346352615723"/>
       <origin rpy="0 0 0" xyz="0 0 0"/>
-      <inertia ixx="0.001488247009527325" ixy="0.0" ixz="0.0" iyy="0.0013525719181349898" iyz="-0.0" izz="0.001488247009527325"/>
+      <inertia ixx="0.000122" ixy="-0.0" ixz="-0.0" iyy="0.000122" iyz="-0.0" izz="0.000137"/>
     </inertial>
     <collision name="right_wheel_collision">
@@ -266,5 +270,8 @@
       <hardwareInterface>hardware_interface/EffortJointInterface</hardwareInterface>
     </joint>
-    <actuator name="right_wheel_motor"/>
+    <actuator name="right_wheel_motor">
+      <hardwareInterface>hardware_interface/EffortJointInterface</hardwareInterface>
+      <mechanicalReduction>1</mechanicalReduction>
+    </actuator>
   </transmission>
   <link name="hokuyo">

Commit message: edge sensor fixes

File: interfearence-description/urdf/cad_interfearence.urdf.xacro (robot description, xacro)
@@ -12,4 +12,29 @@
     <!-- plugin to simulate the electromagnet -->
     <plugin name="magnet" filename="libmagnet_plugin.so"/>
+    <!-- plugins for the edge sensors -->
+    <plugin name="front_left_line_sensor_plugin"
+            filename="libarena_edge_detection_plugin.so">
+        <frameName>/$(arg robotns)/front_left_line_sensor</frameName>
+        <topicName>/$(arg robotns)/edge_sensors/front_left</topicName>
+        <linkName>front_left_line_sensor</linkName>
+    </plugin>
+    <plugin name="front_right_line_sensor_plugin"
+            filename="libarena_edge_detection_plugin.so">
+        <frameName>/$(arg robotns)/front_right_line_sensor</frameName>
+        <topicName>/$(arg robotns)/edge_sensors/front_right</topicName>
+        <linkName>front_right_line_sensor</linkName>
+    </plugin>
+    <plugin name="rear_left_line_sensor_plugin"
+            filename="libarena_edge_detection_plugin.so">
+        <frameName>/$(arg robotns)/rear_left_line_sensor</frameName>
+        <topicName>/$(arg robotns)/edge_sensors/rear_left</topicName>
+        <linkName>rear_left_line_sensor</linkName>
+    </plugin>
+    <plugin name="rear_right_line_sensor_plugin"
+            filename="libarena_edge_detection_plugin.so">
+        <frameName>/$(arg robotns)/rear_right_line_sensor</frameName>
+        <topicName>/$(arg robotns)/edge_sensors/rear_right</topicName>
+        <linkName>rear_right_line_sensor</linkName>
+    </plugin>
     <self_collide>false</self_collide>
   </gazebo>
@@ -77,34 +102,12 @@
   </link>
   <gazebo reference="front_left_line_sensor">
-    <sensor name="front_left_line_sensor_sensor" type="camera">
-      <camera name="front_left_camera">
-        <image>
-          <width>1</width>
-          <height>1</height>
-          <format>R8G8B8</format>
-        </image>
-        <clip>
-          <near>0.002</near>
-        </clip>
-      </camera>
-      <plugin name="front_left_edge_detector_plugin"
-              filename="libarena_edge_detection_plugin.so">
-        <cameraName>front_left_camera</cameraName>
-        <alwaysOn>true</alwaysOn>
-        <updateRate>30</updateRate>
-        <imageTopicName>rgb/image_raw</imageTopicName>
-        <cameraInfoTopicName>rgb/camera_info</cameraInfoTopicName>
-        <frameName>/$(arg robotns)/front_left_line_sensor</frameName>
-        <topicName>/$(arg robotns)/edge_sensors/front_left</topicName>
-        <upperThreshhold>0.52</upperThreshhold>
-        <lowerThreshhold>0.42</lowerThreshhold>
-      </plugin>
-    </sensor>
-    <material>Gazebo/Red</material>
-  </gazebo>
-  <joint name="front_left_line_sensor_joint" type="fixed">
+    <material>Gazebo/Red</material>
+  </gazebo>
+  <joint name="front_left_line_sensor_joint" type="prismatic">
     <parent link="base_footprint"/>
     <child link="front_left_line_sensor"/>
     <origin rpy="0 0 0" xyz="0.08972 -0.05966  0.000631"/>
+    <axis xyz="0 0 1"/>
+    <limit lower="0" upper="0.0001" effort="0" velocity="0"/>
   </joint>
   <link name="front_right_line_sensor">
@@ -127,34 +130,12 @@
   </link>
   <gazebo reference="front_right_line_sensor">
-    <sensor name="front_right_line_sensor_sensor" type="camera">
-      <camera name="front_right_camera">
-        <image>
-          <width>1</width>
-          <height>1</height>
-          <format>R8G8B8</format>
-        </image>
-        <clip>
-          <near>0.002</near>
-        </clip>
-      </camera>
-      <plugin name="front_right_edge_detector_plugin"
-              filename="libarena_edge_detection_plugin.so">
-        <cameraName>front_right_camera</cameraName>
-        <alwaysOn>true</alwaysOn>
-        <updateRate>30</updateRate>
-        <imageTopicName>rgb/image_raw</imageTopicName>
-        <cameraInfoTopicName>rgb/camera_info</cameraInfoTopicName>
-        <frameName>/$(arg robotns)/front_right_line_sensor</frameName>
-        <topicName>/$(arg robotns)/edge_sensors/front_right</topicName>
-        <upperThreshhold>0.52</upperThreshhold>
-        <lowerThreshhold>0.42</lowerThreshhold>
-      </plugin>
-    </sensor>
-    <material>Gazebo/Red</material>
-  </gazebo>
-  <joint name="front_right_line_sensor_joint" type="fixed">
+    <material>Gazebo/Red</material>
+  </gazebo>
+  <joint name="front_right_line_sensor_joint" type="prismatic">
     <parent link="base_footprint"/>
     <child link="front_right_line_sensor"/>
     <origin rpy="0 0 0" xyz="-0.08972 -0.05966  0.000631"/>
+    <axis xyz="0 0 1"/>
+    <limit lower="0" upper="0.0001" effort="0" velocity="0"/>
   </joint>
   <link name="front_scoop">
@@ -346,34 +327,12 @@
   </link>
   <gazebo reference="rear_right_line_sensor">
-    <sensor name="rear_right_line_sensor_sensor" type="camera">
-      <camera name="rear_right_camera">
-        <image>
-          <width>1</width>
-          <height>1</height>
-          <format>R8G8B8</format>
-        </image>
-        <clip>
-          <near>0.002</near>
-        </clip>
-      </camera>
-      <plugin name="rear_right_edge_detector_plugin"
-              filename="libarena_edge_detection_plugin.so">
-        <cameraName>rear_right_camera</cameraName>
-        <alwaysOn>true</alwaysOn>
-        <updateRate>30</updateRate>
-        <imageTopicName>rgb/image_raw</imageTopicName>
-        <cameraInfoTopicName>rgb/camera_info</cameraInfoTopicName>
-        <frameName>/$(arg robotns)/rear_right_line_sensor</frameName>
-        <topicName>/$(arg robotns)/edge_sensors/rear_right</topicName>
-        <upperThreshhold>0.5</upperThreshhold>
-        <lowerThreshhold>0.4</lowerThreshhold>
-      </plugin>
-    </sensor>
-    <material>Gazebo/Red</material>
-  </gazebo>
-  <joint name="rear_right_line_sensor_joint" type="fixed">
+    <material>Gazebo/Red</material>
+  </gazebo>
+  <joint name="rear_right_line_sensor_joint" type="prismatic">
     <parent link="base_footprint"/>
     <child link="rear_right_line_sensor"/>
     <origin rpy="0 0 0" xyz="-0.08925  0.08981  0.00011"/>
+    <axis xyz="0 0 1"/>
+    <limit lower="0" upper="0.0001" effort="0" velocity="0"/>
   </joint>
   <link name="rear_left_line_sensor">
@@ -396,34 +355,12 @@
   </link>
   <gazebo reference="rear_left_line_sensor">
-    <sensor name="rear_left_line_sensor_sensor" type="camera">
-      <camera name="rear_left_camera">
-        <image>
-          <width>1</width>
-          <height>1</height>
-          <format>R8G8B8</format>
-        </image>
-        <clip>
-          <near>0.002</near>
-        </clip>
-      </camera>
-      <plugin name="rear_left_edge_detector_plugin"
-              filename="libarena_edge_detection_plugin.so">
-        <cameraName>rear_left_camera</cameraName>
-        <alwaysOn>true</alwaysOn>
-        <updateRate>30</updateRate>
-        <imageTopicName>rgb/image_raw</imageTopicName>
-        <cameraInfoTopicName>rgb/camera_info</cameraInfoTopicName>
-        <frameName>/$(arg robotns)/rear_left_line_sensor</frameName>
-        <topicName>/$(arg robotns)/edge_sensors/rear_left</topicName>
-        <upperThreshhold>0.5</upperThreshhold>
-        <lowerThreshhold>0.4</lowerThreshhold>
-      </plugin>
-    </sensor>
-    <material>Gazebo/Red</material>
-  </gazebo>
-  <joint name="rear_left_line_sensor_joint" type="fixed">
+    <material>Gazebo/Red</material>
+  </gazebo>
+  <joint name="rear_left_line_sensor_joint" type="prismatic">
     <parent link="base_footprint"/>
     <child link="rear_left_line_sensor"/>
     <origin rpy="0 0 0" xyz="0.08925 0.08981 0.00011"/>
+    <axis xyz="0 0 1"/>
+    <limit lower="0" upper="0.0001" effort="0" velocity="0"/>
   </joint>
 </robot>
