Commit message: Working laser scanner in reality, with calibration step

File: interfearence-description/urdf/hardware_interfearence.urdf.xacro (robot description, xacro)
@@ -313,5 +313,5 @@
     <parent link="base_footprint"/>
     <child link="hokuyo"/>
-    <origin rpy="0 -0.03 -1.57" xyz="-8.000e-05 -3.485e-02  2.744e-02"/>
+    <origin rpy="3.14 0.0 -1.57" xyz="-8.000e-05 -3.485e-02  2.744e-02"/>
   </joint>
   <link name="rear_right_line_sensor">
